File: pinewood_timer/power_management.kicad_sch (KiCad schematic)
At the start: 0 parts

Commit message: worked on schematic more
Other:
- title: 7-SEG-PLACEMENT -> Power management
Changed lines of the file:
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@@
 	(paper "A4")
 	(title_block
-		(title "7-SEG-PLACEMENT")
+		(title "Power management")
 	)
 )
