File: pinewood_timer/seven_seg_display_placement.kicad_sch (KiCad schematic)
At the start: 0 parts

Commit message: worked on the ir sensors and placement display
Parts:
- added M17, M18, M19, M20: N-MOSFET, symbol 2N2907A_NMOS:nMOS
- added R45, R46, R47, R48: 150, symbol Device:R_Small_US
- added R49, R50, R51, R52, R53, R54, R55: 250, symbol Device:R_Small_US
- added U13: 74LS47, symbol 74xx:74LS47
- added U14, U16: SA39-12YWA, Display_7Segment:Sx39-1xxxxx, symbol Display_Character:SA39-12YWA
- added U15, U17: HDSP-7801, Display_7Segment:HDSP-7801, symbol Display_Character:HDSP-7801
Connections:
- new net: R51.1, U13.11 (c)
- new net: R55.1, U13.14 (g)
- new net: R49.1, U13.13 (a)
- new net: R50.1, U13.12 (b)
- new net: R52.1, U13.10 (d)
- new net: R54.1, U13.15 (f)
- new net: R53.1, U13.9 (e)
- new net +3.3V: M19.1 (E), U13.16 (VCC)
- new net A: R49.2, U14.10 (A), U15.10 (A), U16.10 (A), U17.10 (A)
- new net B: R50.2, U14.9 (B), U15.9 (B), U16.9 (B), U17.9 (B)
- new net C: R51.2, U14.8 (C), U15.8 (C), U16.8 (C), U17.8 (C)
- new net D: R52.2, U14.5 (D), U15.5 (D), U16.5 (D), U17.5 (D)
- new net E: R53.2, U14.4 (E), U15.4 (E), U16.4 (E), U17.4 (E)
- new net F: R54.2, U14.2 (F), U15.2 (F), U16.2 (F), U17.2 (F)
- new net G: R55.2, U14.3 (G), U15.3 (G), U16.3 (G), U17.3 (G)
- new net GND: U13.8 (GND)
- new net PA10: U13.2 (C)
- new net PA8: U13.7 (A)
- new net PA9: U13.1 (B)
- new net R45: R45.2, U14.1 (CA), U14.6 (CA)
- new net R46: R46.2, U15.1 (CA), U15.6 (CA)
- new net R47: R47.2, U16.1 (CA), U16.6 (CA)
- new net R48: R48.2, U17.1 (CA), U17.6 (CA)
Other:
- note added: "The segments from A to G of all the 7 segment displays are connected together. The common pins, either common anode or common cathode are used to select which segment will display"

Commit message: edited placement timer schematic since i can never make up my mind
Parts:
- added M21, M22, M23, M24: N-MOSFET, symbol 2N2907A_NMOS:nMOS
- added R56, R57, R58, R59: 150Ω, symbol Device:R_Small_US
- added R60, R61, R62, R63, R64, R65, R66, R67: 47Ω, symbol Device:R_Small_US
- added U12: 74HC138, symbol 74xx:74HC138
- added U18: TLC59210IN, N20, symbol TLC59210IN_SHIFT_REG:TLC59210IN
- added U19, U21: SA39-12YWA, Display_7Segment:Sx39-1xxxxx, symbol Display_Character:SA39-12YWA
- added U20, U22: HDSP-7801, Display_7Segment:HDSP-7801, symbol Display_Character:HDSP-7801
Connections:
- net PA10 is gone; now on net PA6: U13.2 (C)
- net PA8 is gone; now on net PA4: U13.7 (A)
- net PA9 is gone; now on net PA5: U13.1 (B)
- net +3.3V: now also M23.1 (E), U12.16 (VCC), U12.6 (E2), U18.20 (VCC)
- net A: now also R64.2, U19.10 (A), U20.10 (A), U21.10 (A), U22.10 (A)
- net B: now also R63.2, U19.9 (B), U20.9 (B), U21.9 (B), U22.9 (B)
- net C: now also R62.2, U19.8 (C), U20.8 (C), U21.8 (C), U22.8 (C)
- net C3: now also U16.1 (CA), U16.6 (CA), U21.1 (CA), U21.6 (CA)
- net D: now also R61.2, U19.5 (D), U20.5 (D), U21.5 (D), U22.5 (D)
- net E: now also R60.2, U19.4 (E), U20.4 (E), U21.4 (E), U22.4 (E)
- net F: now also R67.2, U19.2 (F), U20.2 (F), U21.2 (F), U22.2 (F)
- net G: now also R66.2, U19.3 (G), U20.3 (G), U21.3 (G), U22.3 (G)
- net GND: now also U12.4 (~{E0}), U12.5 (~{E1}), U12.8 (GND), U18.11 (GND)
- net PA0: now also R45.2
- net PA1: now also R46.2
- net PA2: now also R47.2
- net PA3: now also R48.2
- net R45 renamed C1
- net C1: now also U19.1 (CA), U19.6 (CA); no longer R45.2
- net R46 renamed C2
- net C2: now also U20.1 (CA), U20.6 (CA); no longer R46.2
- removed net R47: R47.2, U16.1 (CA), U16.6 (CA)
- net R48 renamed C4
- net C4: now also U22.1 (CA), U22.6 (CA); no longer R48.2
- new net: R67.1, U18.19 (*Y1)
- new net: R60.1, U18.12 (*Y8)
- new net: R63.1, U18.15 (*Y5)
- new net: R64.1, U18.16 (*Y4)
- new net: R61.1, U18.13 (*Y7)
- new net: R66.1, U18.18 (*Y2)
- new net: R62.1, U18.14 (*Y6)
- new net: R65.1, U18.17 (*Y3)
- new net H: R65.2
- new net PB0: U18.7 (D6)
- new net PB1: U18.5 (D4)
- new net PB10: U12.3 (A2)
- new net PB2: U18.8 (D7)
- new net PB3: U18.2 (D1)
- new net PB4: U18.3 (D2)
- new net PB5: U18.9 (D8)
- new net PB6: U18.6 (D5)
- new net PB7: U18.4 (D3)
- new net PB8: U12.1 (A0)
- new net PB9: U12.2 (A1)
- new net R1: R56.2, U12.15 (~{Y0})
- new net R2: R57.2, U12.14 (~{Y1})
- new net R3: R58.2, U12.13 (~{Y2})
- new net R4: R59.2, U12.12 (~{Y3})
- new net R5: U12.11 (~{Y4})
- new net R6: U12.10 (~{Y5})
- new net R7: U12.9 (~{Y6})
- new net R8: U12.7 (~{Y7})
Other:
- note added: "NOTHING"
- note added: "PB8-10"
- note added: "if i do it this way then all of the code can be set up the same"
- note added: "so this is what i cooked up forgetting that the TDLT5 something was just hooked up inside like the other diagram. so well see where that goes once some more displays arrive for testing"
- moved on the sheet: M17A, M18A, M19A, M20A, R45, R46, R47, R48, R49, R50, R51, R52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

Commit message: finished 2 lane display pcb
Parts:
- U18: footprint N20 -> (none)
Changed lines of the file:
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@@
 			)
 		)
-		(property "Footprint" "N20"
+		(property "Footprint" ""
 			(at 375.92 66.04 0)
 			(effects
