File: pinewood_timer/seven_seg_display_timer.kicad_sch (KiCad schematic)
At the start: 58 parts, among them J2 Conn_01x12_Pin, J3 Conn_01x12_Pin, M1 N-MOSFET, M10 N-MOSFET, M11 N-MOSFET, M12 N-MOSFET, M13 N-MOSFET, M14 N-MOSFET, M15 N-MOSFET, M16 N-MOSFET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

Commit message: finished 2 lane display pcb
Parts:
- removed U7: 74HC138, symbol 74xx:74HC138
- removed U9: TLC59210IN, N20, symbol TLC59210IN_SHIFT_REG:TLC59210IN
- added U1: 74HC138, SN74HC138DR-MUX:SOIC127P600X175-16N, symbol 74xx:74HC138
- added U7: TLC59210IN, TLC59211IPWR-LEDDRIVER:SOP65P640X120-20N, symbol TLC59210IN_SHIFT_REG:TLC59210IN
- M1, M10, M11, M12, M13, M14, M15, M16, M2, M3, M4, M5, M6, M7, M8, M9: footprint (none) -> PMBT2907A_235:TO-236AB_SOT23_NEX-M
- U2, U3, U4, U5: footprint TDCG1060M_VIS -> (none)
- U6: footprint (none) -> SN74HC138DR-MUX:SOIC127P600X175-16N
- U8: footprint N20 -> TLC59211IPWR-LEDDRIVER:SOP65P640X120-20N
Connections:
- net +3.3V: now also U1.16 (VCC), U1.6 (E2), U7.20 (VCC)
- net GND: now also U1.4 (~{E0}), U1.5 (~{E1}), U1.8 (GND), U7.11 (GND)
- net PC0: now also U7.7 (D6)
- net PC1: now also U7.5 (D4)
- net PC10: now also U1.3 (A2)
- net PC2: now also U7.8 (D7)
- net PC3: now also U7.2 (D1)
- net PC4: now also U7.3 (D2)
- net PC5: now also U7.9 (D8)
- net PC6: now also U7.6 (D5)
- net PC7: now also U7.4 (D3)
- net PC8: now also U1.1 (A0)
- net PC9: now also U1.2 (A1)
- net R25: now also U1.15 (~{Y0})
- net R26: now also U1.14 (~{Y1})
- net R27: now also U1.13 (~{Y2})
- net R28: now also U1.12 (~{Y3})
- net R29: now also U1.11 (~{Y4})
- net R30: now also U1.10 (~{Y5})
- net R31: now also U1.9 (~{Y6})
- net R32: now also U1.7 (~{Y7})
- net at R25.1: now also U7.19 (*Y1)
- net at R31.1: now also U7.13 (*Y7)
- net at R26.1: now also U7.18 (*Y2)
- net at R32.1: now also U7.12 (*Y8)
- net at R28.1: now also U7.16 (*Y4)
- net at R29.1: now also U7.15 (*Y5)
- net at R30.1: now also U7.14 (*Y6)
- net at R27.1: now also U7.17 (*Y3)
- no-connect marks 0 -> 20
Other:
- note removed: "NOTHING"
