File: Hardware/pinewood_timer/seven_seg_display_timer.kicad_sch (KiCad schematic)
At the start: 58 parts, among them J2 Conn_01x12_Pin, J3 Conn_01x12_Pin, M1 N-MOSFET, M10 N-MOSFET, M11 N-MOSFET, M12 N-MOSFET, M13 N-MOSFET, M14 N-MOSFET, M15 N-MOSFET, M16 N-MOSFET, M2 N-MOSFET, M3 N-MOSFET, M4 N-MOSFET, M5 N-MOSFET, M6 N-MOSFET, M7 N-MOSFET, M8 N-MOSFET, M9 N-MOSFET, U1 74HC138, U2 TDCR1050M, U3 TDCR1050M, U4 TDCR1050M, U5 TDCR1050M, U6 74HC138, U7 TLC59210IN, U8 TLC59210IN

Commit message: edited schematic.
realized that mux and led driver only saved me 1 pin and added a lot of extra nonsense
Parts:
- M1, M10, M11, M12, M13, M14, M15, M16, M2, M3, M4, M5, M6, M7, M8, M9: footprint PMBT2907A_235:TO-236AB_SOT23_NEX-M -> TO-236AB_SOT23_NEX; symbol 2N2907A_NMOS:nMOS -> pn2907a-smt:PMBT2907A_235
Connections:
- net +3.3V: now also M1.3, M10.3, M11.3, M12.3, M13.3, M14.3, M15.3, M16.3, M2.3, M3.3, M4.3, M5.3, M6.3, M7.3, M8.3, M9.3; no longer M11.1 (E), M13.1 (E), M14.1 (E), M3.1 (E), M5.1 (E), M6.1 (E)
- net C1: now also M1.2
- net C10: now also M10.2
- net C11: now also M11.2
- net C12: now also M12.2
- net C13: now also M13.2
- net C14: now also M14.2
- net C15: now also M15.2
- net C16: now also M16.2
- net C2: now also M2.2
- net C3: now also M3.2
- net C4: now also M4.2
- net C5: now also M5.2
- net C6: now also M6.2
- net C7: now also M7.2
- net C8: now also M8.2
- net C9: now also M9.2
- net at R3.1: now also M3.1
- net at M2.1: now also R2.1
- net at R10.1: now also M10.1
- net at R15.1: now also M15.1
- net at R9.1: now also M9.1
- net at R12.1: now also M12.1
- net at M7.1: now also R7.1
- net at R13.1: now also M13.1
- net at R6.1: now also M6.1
- net at M1.1: now also R1.1
- net at R16.1: now also M16.1
- net at M8.1: now also R8.1
- net at R4.1: now also M4.1
- net at R14.1: now also M14.1
- net at R5.1: now also M5.1
- net at R11.1: now also M11.1
Other:
- moved on the sheet: M1, M10, M11, M12, M13, M14, M15, M16, M2, M3, M4, M5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
