File: Hardware/timer_display_pcb/timer_display_pcb.kicad_sch (KiCad schematic)
At the start: 42 parts, among them J1 Conn_01x13_Socket, M1 N-MOSFET, M2 N-MOSFET, M3 N-MOSFET, M4 N-MOSFET, M5 N-MOSFET, M6 N-MOSFET, M7 N-MOSFET, M8 N-MOSFET, U1 TDCR1050M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

Commit message: edited schematic.
realized that mux and led driver only saved me 1 pin and added a lot of extra nonsense
Other:
- moved on the sheet: D1, J1, R9
