File: mainboard/mainboard.kicad_sch (KiCad schematic)
At the start: 33 parts, among them J1 Conn_01x18_Pin, J4 Conn_01x11_Pin, J5 Conn_01x04_Pin, J6 USB_B_Micro, SW1 SW_SPDT, U10 AMS1117-3.3, U11 STM32L151CBTxA, Y1 16MHz

Commit message: edited schematic.
realized that mux and led driver only saved me 1 pin and added a lot of extra nonsense
Parts:
- removed C1: .1uF, Capacitor_SMD:C_0805_2012Metric_Pad1.18x1.45mm_HandSolder, symbol Device:C_Small
- removed C13, C15: 10pF, symbol Device:C
- removed C14, C16, C17: 100nF, symbol Device:C
- removed C18: 10nF, symbol Device:C
- removed C19, C20: 1uF, symbol Device:C
- removed D5, D6, D7: LED, symbol Device:LED
- removed D8: RED, symbol Device:LED
- removed J4: Conn_01x11_Pin, symbol Connector:Conn_01x11_Pin
- removed J5: Conn_01x04_Pin, symbol Connector:Conn_01x04_Pin
- removed J6: USB_B_Micro, symbol Connector:USB_B_Micro
- removed R41, R43, R44, R68, R69: 1k5, symbol Device:R_US
- removed R42: 10k, symbol Device:R_US
- removed RST_Button1: RESET, Button_Switch_SMD:SW_SPST_CK_RS282G05A3, symbol Connector:Conn_01x02_Pin
- removed U10: AMS1117-3.3, Package_TO_SOT_SMD:SOT-223-3_TabPin2, symbol Regulator_Linear:AMS1117-3.3
- removed U11: STM32L151CBTxA, Package_QFP:LQFP-48_7x7mm_P0.5mm, symbol MCU_ST_STM32L1:STM32L151CBTxA
- added C1, C4, C6, C7: 100nF, symbol Device:C
- added C2: 10uF, symbol Device:C
- added C3, C5: 10pF, symbol Device:C
- added C8: 10nF, symbol Device:C
- added D1: RED, symbol Device:LED
- added J2: Conn_01x11_Pin, symbol Connector:Conn_01x11_Pin
- added J3: Conn_01x04_Pin, symbol Connector:Conn_01x04_Pin
- added J4: USB_B_Micro, symbol Connector:USB_B_Micro
- added R1: 10k, symbol Device:R_US
- added R2, R3: 1k5, symbol Device:R_US
- added U1: STM32L151CBTxA, Package_QFP:LQFP-48_7x7mm_P0.5mm, symbol MCU_ST_STM32L1:STM32L151CBTxA
- added U2: AMS1117-3.3, Package_TO_SOT_SMD:SOT-223-3_TabPin2, symbol Regulator_Linear:AMS1117-3.3
- C10, C9: value 22uF -> 1uF
- C11: value 100nF -> 22uF
- C12: value 10uF -> 22uF
Connections:
- net +3.3V: now also C2.1, C4.1, C6.1, C7.1, D1.2 (A), J3.1 (Pin_1), R2.1, U1.24 (VDD), U1.36 (VDD), U1.48 (VDD), U2.2 (VO)
- net +3.3VA: now also C9.1, C8.1
- net BOOT0: now also R1.2, U1.44 (BOOT0)
- net GND: now also C12.2, C1.2, C3.2, C5.2, C8.2, J3.4 (Pin_4), J4.5 (GND), R3.1, U1.23 (VSS), U1.35 (VSS), U1.47 (VSS), U1.8 (VSSA), U1.9 (VDDA), U2.1 (GND)
- net HSE_IN: now also C3.1, U1.5 (PH0)
- net HSE_OUT: now also C5.1, U1.6 (PH1)
- net NRST: now also C1.1, U1.7 (NRST); no longer C11.1
- net PWR_LED_CATHODE: now also D1.1 (K), R3.2
- net SW_BOOT0: now also R1.1
- net SW_CLK: now also J3.3 (Pin_3), U1.37 (PA14)
- net SW_DIO: now also J3.2 (Pin_2), U1.34 (PA13)
- net USB_D+: now also J4.3 (D+), R2.2, U1.33 (PA12)
- net USB_D-: now also J4.2 (D-), U1.32 (PA11)
- net VBUS: now also C11.1, J4.1 (VBUS), U2.3 (VI); no longer C9.1
- net at J1.18 (Pin_18): now also U1.18 (PB0)
- net at J1.17 (Pin_17): now also U1.19 (PB1)
- net at J1.16 (Pin_16): now also U1.20 (PB2)
- net at J1.8 (Pin_8): now also U1.21 (PB10)
- net at J1.7 (Pin_7): now also U1.22 (PB11)
- net at J1.6 (Pin_6): now also U1.25 (PB12)
- net at J1.5 (Pin_5): now also U1.26 (PB13)
- net at J1.4 (Pin_4): now also U1.27 (PB14)
- net at J1.3 (Pin_3): now also U1.28 (PB15)
- net at J1.15 (Pin_15): now also U1.39 (PB3)
- net at J1.14 (Pin_14): now also U1.40 (PB4)
- net at J1.13 (Pin_13): now also U1.41 (PB5)
- net at J1.12 (Pin_12): now also U1.42 (PB6)
- net at J1.11 (Pin_11): now also U1.43 (PB7)
- net at J1.10 (Pin_10): now also U1.45 (PB8)
- net at J1.9 (Pin_9): now also U1.46 (PB9)
- new net: J2.1 (Pin_1), U1.10 (PA0)
- new net: J2.2 (Pin_2), U1.11 (PA1)
- new net: J2.3 (Pin_3), U1.12 (PA2)
- new net: J2.4 (Pin_4), U1.13 (PA3)
- new net: J2.5 (Pin_5), U1.14 (PA4)
- new net: J2.6 (Pin_6), U1.15 (PA5)
- new net: J2.7 (Pin_7), U1.16 (PA6)
- new net: J2.8 (Pin_8), U1.17 (PA7)
- new net: J2.9 (Pin_9), U1.29 (PA8)
- new net: J2.10 (Pin_10), U1.30 (PA9)
- new net: J2.11 (Pin_11), U1.31 (PA10)
- new net: C2.2, C4.2, C6.2, C7.2
Other:
- removed sheet infared_sensors
- removed sheet seven_seg_display_placement
- removed sheet seven_seg_display_timer
- note added: "3V3 Reg"
- note removed: "(INPUT)"
- note removed: "(OUTPUT)"
- note removed: "4 IR sensors to go under the track. detects if car is above using IR receiver and IR LED. Also has a comparator to make it toggle. might need adc still."
- note removed: "4 sets of 4 7-segment displays. displays time to thousandths. goes at the end of the track."
- note removed: "4 single 7-segment displays. goes above/below time display. should just display place of each lane."
- note removed: "LANE PLACEMENT"
- note removed: "MUX"
- note removed: "PA10-14 input to read if car/not"
- note removed: "PC0-7 output shift reg PC8-10 mux PB0-7 output shift reg PB8-10 mux"
- note removed: "RESET Button"
- note removed: "SENSORS"
- note removed: "SHIFT REG"
- note removed: "TIME DISPLAY LANES 1-2"
- note removed: "TIME DISPLAY LANES 3-4"
- note removed: "i want to have a large reset button that is accessible to reset the track each run. i also want to have one on the board for funzies"
- note removed: "status leds? *red - rebooting *green - ready *amber - timing?"
