File: display_15_in/tim_disp.kicad_sch (KiCad schematic)
At the start: 56 parts, among them M1 N-MOSFET, M10 N-MOSFET, M11 N-MOSFET, M12 N-MOSFET, M13 N-MOSFET, M14 N-MOSFET, M15 N-MOSFET, M16 N-MOSFET, M2 N-MOSFET, M3 N-MOSFET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

Commit message: added full end of track display board
Parts:
- R1, R11, R12, R16, R17, R18, R19, R2, R20, R21, R22, R23, R26, R27, R28, R3, R31, R32, R4, R5, R6, R7: footprint (none) -> Resistor_SMD:R_0805_2012Metric
- R10: renamed from R8; footprint (none) -> Resistor_SMD:R_0805_2012Metric
- R13: renamed from R14; footprint (none) -> Resistor_SMD:R_0805_2012Metric
- R14: renamed from R15; footprint (none) -> Resistor_SMD:R_0805_2012Metric
- R15: renamed from R13; footprint (none) -> Resistor_SMD:R_0805_2012Metric
- R24: renamed from R25; footprint (none) -> Resistor_SMD:R_0805_2012Metric
- R25: renamed from R24; footprint (none) -> Resistor_SMD:R_0805_2012Metric
- R29: renamed from R30; footprint (none) -> Resistor_SMD:R_0805_2012Metric
- R30: renamed from R29; footprint (none) -> Resistor_SMD:R_0805_2012Metric
- R8: renamed from R9; footprint (none) -> Resistor_SMD:R_0805_2012Metric
- R9: renamed from R10; footprint (none) -> Resistor_SMD:R_0805_2012Metric
- T1: renamed from U1; footprint (none) -> TDCR1050M-4-7-seg-display:TDCG1060M_VIS
- T2: renamed from U4; footprint (none) -> TDCR1050M-4-7-seg-display:TDCG1060M_VIS
- T3: renamed from U5; footprint (none) -> TDCR1050M-4-7-seg-display:TDCG1060M_VIS
- T4: renamed from U8; footprint (none) -> TDCR1050M-4-7-seg-display:TDCG1060M_VIS
- renumbered U2 to U1, U3 to U2, U6 to U3, U7 to U4
Connections:
- net A: now also T1.14, T2.14; no longer T1.16, T2.16
- net A2: now also T3.14, T4.14; no longer T3.16, T4.16
- net B: now also T1.16, T2.16; no longer T1.15, T2.15
- net B2: now also T3.16, T4.16; no longer T3.15, T4.15
- net C: now also T1.13, T2.13; no longer T1.14, T2.14
- net C2: now also T3.13, T4.13; no longer T3.14, T4.14
- net D: now also T1.3, T2.3; no longer T1.13, T2.13
- net D2: now also T3.3, T4.3; no longer T3.13, T4.13
- net E: now also T1.5, T2.5; no longer T1.11, T2.11
- net E2: now also T3.5, T4.5; no longer T3.11, T4.11
- net F: now also T1.11, T2.11; no longer T1.3, T2.3
- net F2: now also T3.11, T4.11; no longer T3.3, T4.3
- net G: now also T1.15, T2.15; no longer T1.5, T2.5
- net G2: now also T3.15, T4.15; no longer T3.5, T4.5
- net H renamed DP1
- net H2 renamed DP2
Other:
- title: (none) -> Time Display
- moved on the sheet: M1, M10, M11, M12, M13, M14, M15, M16, M2, M3, M4, M5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
