File: Hardware/display_15_in/tim_disp.kicad_sch (KiCad schematic)
At the start: 56 parts, among them M1 N-MOSFET, M10 N-MOSFET, M11 N-MOSFET, M12 N-MOSFET, M13 N-MOSFET, M14 N-MOSFET, M15 N-MOSFET, M16 N-MOSFET, M2 N-MOSFET, M3 N-MOSFET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

Commit message: routed more traces
Connections:
- net C2: no longer R26.2, T3.13, T4.13
- new net C_2: R26.2, T3.13, T4.13
Changed lines of the file:
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@@
 		)
 	)
-	(label "C2"
+	(label "C_2"
 		(at 347.969 21.59 0)
 		(effects
@@
 		)
 	)
-	(label "C2"
+	(label "C_2"
 		(at 334.01 167.64 270)
 		(effects
