File: Hardware/display_15_in/display_15_in.kicad_pcb (KiCad board)
At the start: 2 copper layers, 330.2 x 96.5 mm, 78 parts, among them J1 559592430, M1 N-MOSFET, M10 N-MOSFET, M11 N-MOSFET, M12 N-MOSFET, M13 N-MOSFET, M14 N-MOSFET, M15 N-MOSFET, M16 N-MOSFET, M17 N-MOSFET, M18 N-MOSFET, M19 N-MOSFET, M2 N-MOSFET, M20 N-MOSFET, M3 N-MOSFET, M4 N-MOSFET, M5 N-MOSFET, M6 N-MOSFET, M7 N-MOSFET, M8 N-MOSFET, M9 N-MOSFET, T1 TDCR1050M, T2 TDCR1050M, T3 TDCR1050M, T4 TDCR1050M, U1 74HC138, U2 TLC59210IN, U3 74HC138, U4 TLC59210IN, U5 SA39-12YWA, U6 SA39-12YWA, U7 SA39-12YWA, U8 SA39-12YWA, U9 S16B-PHDSSLFSN

Commit message: more work on pcb
finished house season 2 and made decent progress (i think) on the pcb. if it is bad ill see tomorrow lol
Parts:
- moved R33 35.1 mm to (303.7, 261.1), turned to 0 degrees
- moved M17 34.9 mm to (303.8, 265.2), turned to -90 degrees
- moved R14 18.9 mm to (340.4, 311.3), turned to 90 degrees
- moved R11 17.4 mm to (344.4, 311.3), turned to 90 degrees
- moved R30 17.2 mm to (522.5, 312.5)
- moved R32 17.0 mm to (518.4, 312.5)
- moved R27 16.8 mm to (494.0, 312.5)
- moved R7 14.3 mm to (324.1, 311.4), turned to 90 degrees
- moved R13 13.2 mm to (316.0, 311.5)
- moved M19 12.7 mm to (445.0, 272.9)
- moved R12 12.5 mm to (336.3, 311.3), turned to 90 degrees
- moved R35 9.63 mm to (445.1, 277.4), turned to 180 degrees
- moved R9 9.58 mm to (328.2, 311.4), turned to 90 degrees
- moved R25 9.22 mm to (506.2, 312.5)
- moved R16 9.19 mm to (320.0, 311.4), turned to 90 degrees
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Routing:
- net PA0: track 0.00 -> 307.0 mm, vias 0 -> 3
- net PA1: track 0.00 -> 304.3 mm, vias 0 -> 6
- net PA2: track 0.00 -> 300.2 mm, vias 0 -> 4
- net PA6: track 0.00 -> 219.3 mm, vias 0 -> 4
- net PA3: track 0.00 -> 219.2 mm, vias 0 -> 2
- net PA5: track 0.00 -> 219.0 mm, vias 0 -> 4
- net PA4: track 0.00 -> 218.2 mm, vias 0 -> 4
- net /tim_disp/C2: track 0.00 -> 122.5 mm, vias 0 -> 2
- net /tim_disp/A2: track 0.00 -> 115.1 mm, vias 0 -> 2
- net /tim_disp/G2: track 0.00 -> 115.0 mm, vias 0 -> 2
- net PA7: track 0.00 -> 114.3 mm, vias 0 -> 2
- net /tim_disp/D2: track 0.00 -> 114.2 mm, vias 0 -> 4
- net /tim_disp/E2: track 0.00 -> 113.8 mm, vias 0 -> 3
- net /tim_disp/B2: track 0.00 -> 113.4 mm, vias 0 -> 2
- net /tim_disp/F2: track 0.00 -> 111.9 mm, vias 0 -> 4
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Other:
- board size 330.2 x 96.5 mm -> 330.2 x 100.3 mm

Commit message: routed more traces
Routing:
- net PC9: track 0.00 -> 124.1 mm, vias 0 -> 2
- net PA3: track 219.2 -> 320.5 mm, vias 2 -> 4
- net PA4: track 218.2 -> 317.4 mm, vias 4 -> 6
- net PA6: track 219.3 -> 316.5 mm, vias 4 -> 6
- net PA5: track 219.0 -> 314.6 mm
- net PC5: track 5.35 -> 87.8 mm, vias 0 -> 2
- net /tim_disp/R8: track 0.00 -> 82.2 mm, vias 0 -> 2
- net PB8: track 0.00 -> 37.3 mm, vias 0 -> 1
- net PB10: track 0.00 -> 33.6 mm, vias 0 -> 1
- net PB9: track 7.82 -> 25.5 mm, vias 0 -> 1
- net PC8: track 0.00 -> 10.4 mm, vias 0 -> 2
- net +3.3V: track 0.00 -> 10.4 mm
- net PC10: track 0.00 -> 8.40 mm, vias 0 -> 2
- net PB3: track 7.55 -> 10.8 mm, vias 0 -> 1
- net PB6: track 92.6 -> 93.5 mm
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
Commit message: added more traces lowkey sufferig
Parts:
- moved R11 28.5 mm to (316.0, 312.4)
- moved R13 28.5 mm to (344.4, 312.2)
- moved R14 20.3 mm to (320.0, 312.4)
- moved R16 20.3 mm to (340.4, 312.3)
- moved R12 12.2 mm to (324.1, 312.4)
- moved R7 12.2 mm to (336.3, 312.3)
- moved R8 4.16 mm to (328.2, 312.3)
- moved R9 4.16 mm to (332.2, 312.3)
Routing:
- net PA14: track 40.9 -> 249.9 mm, vias 2 -> 3
- net PA11: track 58.6 -> 212.5 mm, vias 2 -> 6
- net PC10: track 8.40 -> 143.4 mm, vias 2 -> 3
- net PC8: track 10.4 -> 133.9 mm, vias 2 -> 3
- net /tim_disp/A: track 0.00 -> 115.1 mm, vias 0 -> 2
- net /tim_disp/G: track 0.00 -> 115.0 mm, vias 0 -> 2
- net /tim_disp/D: track 0.00 -> 114.2 mm, vias 0 -> 4
- net /tim_disp/C: track 0.00 -> 113.9 mm, vias 0 -> 2
- net /tim_disp/E: track 0.00 -> 113.8 mm, vias 0 -> 3
- net /tim_disp/B: track 0.00 -> 113.4 mm, vias 0 -> 2
- net /tim_disp/F: track 0.00 -> 111.9 mm, vias 0 -> 4
- net PA13: track 46.2 -> 156.1 mm, vias 2 -> 5
- net PB9: track 25.5 -> 135.0 mm
- net /tim_disp/DP1: track 0.00 -> 103.2 mm, vias 0 -> 2
- net PB8: track 37.3 -> 130.8 mm
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Other:
- board size 330.2 x 100.3 mm -> 330.2 x 102.9 mm

Commit message: avoiding doing the via calculations or at least researching how to do them so i just added silkscreen stuff
Other:
- board text added: "74HC138"
- board text added: "PT204-6B"
- board text added: "TLC59210IN"
Changed lines of the file:
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@@
 		(at 342.9 335.28 180)
 		(property "Reference" "U2"
-			(at -0.325 -4.385 0)
+			(at 0 -4.385 0)
 			(layer "F.SilkS")
 			(effects
@@
 		(at 495.3 335.28)
 		(property "Reference" "U4"
-			(at -0.325 -4.385 0)
+			(at 0 4.572 0)
 			(layer "F.SilkS")
 			(effects
@@
 		(layer "User.4")
 	)
+	(gr_text "TLC59210IN"
+		(at 490.728 331.216 0)
+		(layer "F.SilkS")
+		(effects
+			(font
+				(size 1 1)
+				(thickness 0.1)
+			)
+			(justify left bottom)
+		)
+	)
+	(gr_text "PT204-6B"
+		(at 548.64 350.52 0)
+		(layer "F.SilkS")
+		(effects
+			(font
+				(size 1 1)
+				(thickness 0.1)
+			)
+			(justify left bottom)
+		)
+	)
+	(gr_text "74HC138"
+		(at 324.612 338.836 90)
+		(layer "F.SilkS")
+		(effects
+			(font
+				(size 1 1)
+				(thickness 0.1)
+			)
+			(justify left bottom)
+		)
+	)
+	(gr_text "74HC138"
+		(at 527.812 338.836 90)
+		(layer "F.SilkS")
+		(effects
+			(font
+				(size 1 1)
+				(thickness 0.1)
+			)
+			(justify left bottom)
+		)
+	)
+	(gr_text "TLC59210IN"
+		(at 338.328 330.2 0)
+		(layer "F.SilkS")
+		(effects
+			(font
+				(size 1 1)
+				(thickness 0.1)
+			)
+			(justify left bottom)
+		)
+	)
+	(gr_text "PT204-6B"
+		(at 281.94 350.52 0)
+		(layer "F.SilkS")
+		(effects
+			(font
+				(size 1 1)
+				(thickness 0.1)
+			)
+			(justify left bottom)
+		)
+	)
+	(gr_text "PT204-6B"
+		(at 370.84 350.012 0)
+		(layer "F.SilkS")
+		(effects
+			(font
+				(size 1 1)
+				(thickness 0.1)
+			)
+			(justify left bottom)
+		)
+	)
+	(gr_text "PT204-6B"
+		(at 459.74 350.012 0)
+		(layer "F.SilkS")
+		(effects
+			(font
+				(size 1 1)
+				(thickness 0.1)
+			)
+			(justify left bottom)
+		)
+	)
 	(gr_text "empty"
 		(at 297.18 132.08 0)
@@
 	)
 	(via
-		(at 498.094 339.598)
+		(at 499.968244 338.215099)
 		(size 0.6)
 		(drill 0.3)
