File: Hardware/display_15_in/display_15_in.kicad_pcb (KiCad board)
At the start: 2 copper layers, 330.2 x 106.7 mm, 78 parts, among them J1 559592430, M1 N-MOSFET, M10 N-MOSFET, M11 N-MOSFET, M12 N-MOSFET, M13 N-MOSFET, M14 N-MOSFET, M15 N-MOSFET, M16 N-MOSFET, M17 N-MOSFET, M18 N-MOSFET, M19 N-MOSFET, M2 N-MOSFET, M20 N-MOSFET, M3 N-MOSFET, M4 N-MOSFET, M5 N-MOSFET, M6 N-MOSFET, M7 N-MOSFET, M8 N-MOSFET, M9 N-MOSFET, T1 TDCR1050M, T2 TDCR1050M, T3 TDCR1050M, T4 TDCR1050M, U1 74HC138, U2 TLC59210IN, U3 74HC138, U4 TLC59210IN, U5 SA39-12YWA, U6 SA39-12YWA, U7 SA39-12YWA, U8 SA39-12YWA, U9 S16B-PHDSSLFSN

Commit message: began work on mainboard
mostly schematic but i did assign footprints (if you even consider that to be working on the pcb)
power in from usb and ONLY power from usb - no dp just vbus and gnd. still dnt know what cc or shield is but i can figure that out later
jtag and usb-ttl for programming. will not be powered by usb while programmed.
Parts:
- added 3V1: TestPoint, TestPoint:TestPoint_Keystone_5019_Minature, B.Cu at (269.0, 337.8)
- added 3V2: TestPoint, TestPoint:TestPoint_Keystone_5019_Minature, B.Cu at (542.8, 355.3)
- added 3V3: TestPoint, TestPoint:TestPoint_Keystone_5019_Minature, B.Cu at (441.7, 320.5)
- added 3V4: TestPoint, TestPoint:TestPoint_Keystone_5019_Minature, F.Cu at (400.1, 342.9)
- added GND1: TestPoint, TestPoint:TestPoint_Keystone_5019_Minature, F.Cu at (571.5, 336.6)
- added GND2: TestPoint, TestPoint:TestPoint_Keystone_5019_Minature, F.Cu at (266.7, 336.6)
- added GND3: TestPoint, TestPoint:TestPoint_Keystone_5019_Minature, B.Cu at (309.9, 275.1)
- added GND4: TestPoint, TestPoint:TestPoint_Keystone_5019_Minature, B.Cu at (508.0, 274.3)
- added GND5: TestPoint, TestPoint:TestPoint_Keystone_5019_Minature, F.Cu at (502.9, 350.5)
- added GND6: TestPoint, TestPoint:TestPoint_Keystone_5019_Minature, F.Cu at (508.0, 273.1)
- added GND7: TestPoint, TestPoint:TestPoint_Keystone_5019_Minature, F.Cu at (330.2, 273.1)
- added GND8: TestPoint, TestPoint:TestPoint_Keystone_5019_Minature, F.Cu at (400.1, 337.8)
- added PA11: TP, TestPoint:TestPoint_Keystone_5019_Minature, F.Cu at (390.2, 297.0)
- added PA12: TP, TestPoint:TestPoint_Keystone_5019_Minature, F.Cu at (397.7, 297.0)
- added PA13: TP, TestPoint:TestPoint_Keystone_5019_Minature, F.Cu at (408.9, 297.0)
- added PA14: TP, TestPoint:TestPoint_Keystone_5019_Minature, F.Cu at (420.4, 292.1)
- renumbered R18 to R10, R19 to R11, R20 to R12, R21 to R13, R22 to R14, R24 to R15, R29 to R16, R7 to R17, R8 to R18, R9 to R19, R11 to R20, R12 to R21, R13 to R22, R14 to R23, R16 to R24, R23 to R25, R25 to R26, R26 to R27, R27 to R28, R28 to R29, R10 to R7, R15 to R8, R17 to R9, U9 to U1, U4 to U3, U1 to U4, U3 to U5, U5 to U6, U6 to U7, U7 to U8, U8 to U9
Routing:
- net PA13: track 156.2 -> 161.8 mm
- net PA11: track 212.5 -> 217.8 mm
- net PA12: track 131.3 -> 135.0 mm
- net PA14: track 248.9 -> 251.8 mm

Commit message: display and design rules
Parts:
- moved 3V2 265.6 mm to (342.3, 181.2)
- moved 3V3 265.6 mm to (241.2, 146.4)
- moved 3V4 265.6 mm to (199.5, 168.7)
- moved GND1 265.6 mm to (371.0, 162.4)
- moved GND2 265.6 mm to (66.2, 162.4)
- moved GND3 265.6 mm to (109.3, 100.9)
- moved GND4 265.6 mm to (307.5, 100.2)
- moved GND5 265.6 mm to (302.4, 176.4)
- moved GND6 265.6 mm to (307.5, 98.9)
- moved GND7 265.6 mm to (129.7, 98.9)
- moved GND8 265.6 mm to (199.5, 163.7)
- moved J1 265.6 mm to (229.6, 168.7)
- moved M1 265.6 mm to (79.9, 146.2)
- moved M10 265.6 mm to (250.1, 146.4)
- moved M11 265.6 mm to (272.9, 146.4)
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Routing:
- net +3.3V: track 701.1 -> 709.7 mm
- net Net-(U3-*Y7): track 29.3 -> 30.5 mm
- net Net-(U3-*Y1): track 33.3 -> 34.0 mm
- net Net-(U3-*Y8): track 35.5 -> 36.2 mm
Other:
- copper layers 2 -> 4
- board text removed: "empty"
- board text removed: "track"

Commit message: lowkey accidentally deleted everything but i brought a previous commit back since i am a true girlboss
like i deleted inner layers since i thought iw as looking at a diff board
Parts:
- added REF**: MountingHole_4.3mm_M4, MountingHole:MountingHole_4.3mm_M4, F.Cu at (373.8, 174.1)
- added REF**: MountingHole_4.3mm_M4, MountingHole:MountingHole_4.3mm_M4, F.Cu at (373.9, 87.1)
- added REF**: MountingHole_4.3mm_M4, MountingHole:MountingHole_4.3mm_M4, F.Cu at (218.4, 130.8)
- added REF**: MountingHole_4.3mm_M4, MountingHole:MountingHole_4.3mm_M4, F.Cu at (63.3, 174.1)
- added REF**: MountingHole_4.3mm_M4, MountingHole:MountingHole_4.3mm_M4, F.Cu at (63.2, 87.1)
- M2: value N-MOSFET -> PN2907A
- moved 3V1 3.35 mm to (68.6, 167.0)
- turned PA11 to 0 degrees
Routing:
- net PA13: track 161.8 -> 162.6 mm
Other:
- copper layers 4 -> 2
- board text added: "150Ω"
- board text added: "47Ω"
- board text added: "56KΩ"
- board text added: "PN2907A"

Commit message: final push for the night
Parts:
- added G***: LOGO, LOGO, F.Cu at (218.4, 144.8)
Other:
- board text added: "REV 1"
- board text added: "Timer Display Board"

Commit message: generated gbr files
Changed lines of the file:
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@@
 			(at 0 -5.3 0)
 			(layer "F.SilkS")
+			(hide yes)
 			(effects
 				(font
@@
 			(at 0 -5.3 90)
 			(layer "F.SilkS")
+			(hide yes)
 			(effects
 				(font
@@
 			(at 0 -5.3 90)
 			(layer "F.SilkS")
+			(hide yes)
 			(effects
 				(font
@@
 			(at 0 -5.3 0)
 			(layer "F.SilkS")
+			(hide yes)
 			(effects
 				(font
