File: Hardware/display_15_in/_autosave-display_15_in.kicad_pcb (KiCad board)
At the start: 2 copper layers, 330.2 x 106.7 mm, 78 parts, among them J1 559592430, M1 N-MOSFET, M10 N-MOSFET, M11 N-MOSFET, M12 N-MOSFET, M13 N-MOSFET, M14 N-MOSFET, M15 N-MOSFET, M16 N-MOSFET, M17 N-MOSFET, M18 N-MOSFET, M19 N-MOSFET, M2 N-MOSFET, M20 N-MOSFET, M3 N-MOSFET, M4 N-MOSFET, M5 N-MOSFET, M6 N-MOSFET, M7 N-MOSFET, M8 N-MOSFET, M9 N-MOSFET, T1 TDCR1050M, T2 TDCR1050M, T3 TDCR1050M, T4 TDCR1050M, U1 74HC138, U2 TLC59210IN, U3 74HC138, U4 TLC59210IN, U5 SA39-12YWA, U6 SA39-12YWA, U7 SA39-12YWA, U8 SA39-12YWA, U9 S16B-PHDSSLFSN

Commit message: power traces, gnd plane vias, and test points
Parts:
- added TP1: TestPoint, TestPoint:TestPoint_Keystone_5019_Minature, B.Cu at (269.0, 337.8)
- added TP10: TestPoint, TestPoint:TestPoint_Keystone_5019_Minature, F.Cu at (508.0, 273.1)
- added TP11: TestPoint, TestPoint:TestPoint_Keystone_5019_Minature, F.Cu at (323.9, 273.1)
- added TP12: TestPoint, TestPoint:TestPoint_Keystone_5019_Minature, F.Cu at (400.1, 337.8)
- added TP13: TP, TestPoint:TestPoint_Keystone_5019_Minature, F.Cu at (390.2, 297.0)
- added TP14: TP, TestPoint:TestPoint_Keystone_5019_Minature, F.Cu at (397.7, 297.0)
- added TP15: TP, TestPoint:TestPoint_Keystone_5019_Minature, F.Cu at (408.9, 297.2)
- added TP16: TP, TestPoint:TestPoint_Keystone_5019_Minature, F.Cu at (420.4, 292.1)
- added TP2: TestPoint, TestPoint:TestPoint_Keystone_5019_Minature, B.Cu at (542.8, 355.3)
- added TP3: TestPoint, TestPoint:TestPoint_Keystone_5019_Minature, B.Cu at (441.7, 320.5)
- added TP4: TestPoint, TestPoint:TestPoint_Keystone_5019_Minature, F.Cu at (400.1, 342.9)
- added TP5: TestPoint, TestPoint:TestPoint_Keystone_5019_Minature, F.Cu at (336.6, 237.5)
- added TP6: TestPoint, TestPoint:TestPoint_Keystone_5019_Minature, F.Cu at (306.1, 225.6)
- added TP7: TestPoint, TestPoint:TestPoint_Keystone_5019_Minature, B.Cu at (309.9, 275.1)
- added TP8: TestPoint, TestPoint:TestPoint_Keystone_5019_Minature, B.Cu at (508.0, 274.3)
- added TP9: TestPoint, TestPoint:TestPoint_Keystone_5019_Minature, F.Cu at (502.9, 350.5)
- renumbered R18 to R10, R19 to R11, R20 to R12, R21 to R13, R22 to R14, R24 to R15, R29 to R16, R7 to R17, R8 to R18, R9 to R19, R11 to R20, R12 to R21, R13 to R22, R14 to R23, R16 to R24, R23 to R25, R25 to R26, R26 to R27, R27 to R28, R28 to R29, R10 to R7, R15 to R8, R17 to R9, U9 to U1, U4 to U3, U1 to U4, U3 to U5, U5 to U6, U6 to U7, U7 to U8, U8 to U9
Routing:
- net PA13: track 156.2 -> 161.8 mm
- net PA11: track 212.5 -> 217.8 mm
- net PA12: track 131.3 -> 135.0 mm
- net PA14: track 248.9 -> 251.8 mm
