File: Hardware/display_15_in/plc_disp.kicad_sch (KiCad schematic)
At the start: 12 parts, among them M17 N-MOSFET, M18 N-MOSFET, M19 N-MOSFET, M20 N-MOSFET, U5 SA39-12YWA, U6 SA39-12YWA, U7 SA39-12YWA, U8 SA39-12YWA

Commit message: power traces, gnd plane vias, and test points
Parts:
- renumbered U5 to U6, U6 to U7, U7 to U8, U8 to U9
Connections:
- net C1 renamed CA1
- net C2 renamed CA2
- net C3 renamed CA3
- net C4 renamed CA4
Changed lines of the file:
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@@
 	(wire
 		(pts
-			(xy 140.97 64.77) (xy 140.97 60.96)
+			(xy 140.97 60.96) (xy 140.97 64.77)
 		)
 		(stroke
@@
 		)
 	)
-	(label "C3"
-		(at 111.76 60.96 0)
-		(effects
-			(font
-				(size 1.27 1.27)
-			)
-			(justify left bottom)
-		)
-	)
-	(label "C1"
+	(label "CA1"
 		(at 48.26 60.96 0)
 		(effects
@@
 		)
 	)
-	(label "C3"
-		(at 115.57 53.34 0)
+	(label "CA1"
+		(at 52.07 50.8 0)
 		(effects
 			(font
@@
 		)
 	)
-	(label "C4"
+	(label "CA4"
 		(at 140.97 60.96 0)
+		(effects
+			(font
+				(size 1.27 1.27)
+			)
+			(justify left bottom)
+		)
+	)
+	(label "CA3"
+		(at 111.76 60.96 0)
 		(effects
 			(font
@@
 		)
 	)
+	(label "CA3"
+		(at 115.57 50.8 0)
+		(effects
+			(font
+				(size 1.27 1.27)
+			)
+			(justify left bottom)
+		)
+	)
 	(label "A"
 		(at 127 24.13 0)
@@
 		)
 	)
+	(label "CA2"
+		(at 80.01 60.96 0)
+		(effects
+			(font
+				(size 1.27 1.27)
+			)
+			(justify left bottom)
+		)
+	)
 	(label "G"
 		(at 119.38 16.51 0)
@@
 		)
 	)
+	(label "CA4"
+		(at 144.78 50.8 0)
+		(effects
+			(font
+				(size 1.27 1.27)
+			)
+			(justify left bottom)
+		)
+	)
 	(label "P_SEL_4"
 		(at 128.27 69.85 180)
@@
 		)
 	)
-	(label "C4"
-		(at 144.78 53.34 0)
-		(effects
-			(font
-				(size 1.27 1.27)
-			)
-			(justify left bottom)
-		)
-	)
 	(label "E"
 		(at 121.92 19.05 0)
@@
 		)
 	)
-	(label "C2"
-		(at 80.01 60.96 0)
-		(effects
-			(font
-				(size 1.27 1.27)
-			)
-			(justify left bottom)
-		)
-	)
-	(label "C2"
-		(at 83.82 53.34 0)
-		(effects
-			(font
-				(size 1.27 1.27)
-			)
-			(justify left bottom)
-		)
-	)
-	(label "C1"
-		(at 52.07 53.34 0)
-		(effects
-			(font
-				(size 1.27 1.27)
-			)
-			(justify left bottom)
-		)
-	)
 	(label "C"
 		(at 124.46 21.59 0)
+		(effects
+			(font
+				(size 1.27 1.27)
+			)
+			(justify left bottom)
+		)
+	)
+	(label "CA2"
+		(at 83.82 50.8 0)
 		(effects
 			(font
@@
 		(dnp no)
 		(fields_autoplaced yes)
-		(property "Reference" "U6"
+		(property "Reference" "U7"
 			(at 74.93 25.4 0)
 			(effects
@@
 			(project "display_15_in"
 				(path "/78ee3e98-fb3d-4210-9692-4d335f53f951/50e4659a-a69d-4e7c-9e84-cd1a86a745dc"
-					(reference "U6")
+					(reference "U7")
 					(unit 1)
 				)
@@
 		(on_board yes)
 		(dnp no)
-		(property "Reference" "#PWR032"
+		(property "Reference" "#PWR046"
 			(at 140.97 83.8602 0)
 			(effects
@@
 			(project "display_15_in"
 				(path "/78ee3e98-fb3d-4210-9692-4d335f53f951/50e4659a-a69d-4e7c-9e84-cd1a86a745dc"
-					(reference "#PWR032")
+					(reference "#PWR046")
 					(unit 1)
 				)
@@
 		(dnp no)
 		(fields_autoplaced yes)
-		(property "Reference" "U5"
+		(property "Reference" "U6"
 			(at 43.18 25.4 0)
 			(effects
@@
 			(project "display_15_in"
 				(path "/78ee3e98-fb3d-4210-9692-4d335f53f951/50e4659a-a69d-4e7c-9e84-cd1a86a745dc"
-					(reference "U5")
+					(reference "U6")
 					(unit 1)
 				)
@@
 		(on_board yes)
 		(dnp no)
-		(property "Reference" "#PWR031"
+		(property "Reference" "#PWR045"
 			(at 111.76 83.82 0)
 			(effects
@@
 			(project "display_15_in"
 				(path "/78ee3e98-fb3d-4210-9692-4d335f53f951/50e4659a-a69d-4e7c-9e84-cd1a86a745dc"
-					(reference "#PWR031")
+					(reference "#PWR045")
 					(unit 1)
 				)
@@
 		(on_board yes)
 		(dnp no)
-		(property "Reference" "#PWR030"
+		(property "Reference" "#PWR044"
 			(at 80.01 83.82 0)
 			(effects
@@
 			(project "display_15_in"
 				(path "/78ee3e98-fb3d-4210-9692-4d335f53f951/50e4659a-a69d-4e7c-9e84-cd1a86a745dc"
-					(reference "#PWR030")
+					(reference "#PWR044")
 					(unit 1)
 				)
@@
 		(dnp no)
 		(fields_autoplaced yes)
-		(property "Reference" "U8"
+		(property "Reference" "U9"
 			(at 135.89 25.4 0)
 			(effects
@@
 			(project "display_15_in"
 				(path "/78ee3e98-fb3d-4210-9692-4d335f53f951/50e4659a-a69d-4e7c-9e84-cd1a86a745dc"
-					(reference "U8")
+					(reference "U9")
 					(unit 1)
 				)
@@
 		(on_board yes)
 		(dnp no)
-		(property "Reference" "#PWR029"
+		(property "Reference" "#PWR043"
 			(at 48.26 83.82 0)
 			(effects
@@
 			(project "display_15_in"
 				(path "/78ee3e98-fb3d-4210-9692-4d335f53f951/50e4659a-a69d-4e7c-9e84-cd1a86a745dc"
-					(reference "#PWR029")
+					(reference "#PWR043")
 					(unit 1)
 				)
@@
 		(dnp no)
 		(fields_autoplaced yes)
-		(property "Reference" "U7"
+		(property "Reference" "U8"
 			(at 106.68 25.4 0)
 			(effects
@@
 			(project "display_15_in"
 				(path "/78ee3e98-fb3d-4210-9692-4d335f53f951/50e4659a-a69d-4e7c-9e84-cd1a86a745dc"
-					(reference "U7")
+					(reference "U8")
 					(unit 1)
 				)
