File: Hardware/mainboard/stm.kicad_sch (KiCad schematic)
At the start: 44 parts, among them J5 race start, SW1 ON-BOARD, SW2 BOT, SW3 BOOT, SW4 SW_SPST, U3 STM32F091RCTx, Y1 Crystal_GND24

Commit message: routed traces
Connections:
- no-connect marks 5 -> 6
Changed lines of the file:
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@@
+	)
+	(no_connect
+		(at 81.28 49.53)
 	)
 	(no_connect

Commit message: fixed schematic pcb agreement errors
Connections:
- net IR_1 renamed LANE_1_IR
- net IR_2 renamed LANE_2_IR
- net IR_3 renamed LANE_3_IR
- net IR_4 renamed LANE_4_IR
Changed lines of the file:
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@@
-		)
-	)
-	(global_label "IR_1"
-		(shape input)
-		(at 190.5 81.28 180)
-		(fields_autoplaced yes)
-		(effects
-			(font
-				(size 1.016 1.016)
-			)
-			(justify right)
-		)
-		(property "Intersheetrefs" "${INTERSHEET_REFS}"
-			(at 184.8706 81.28 0)
-			(effects
-				(font
-					(size 1.27 1.27)
-				)
-				(justify right)
-				(hide yes)
-			)
 		)
 	)
@@
 		)
 	)
-	(global_label "IR_2"
-		(shape input)
-		(at 203.2 81.28 180)
-		(fields_autoplaced yes)
-		(effects
-			(font
-				(size 1.016 1.016)
-			)
-			(justify right)
-		)
-		(property "Intersheetrefs" "${INTERSHEET_REFS}"
-			(at 197.5706 81.28 0)
-			(effects
-				(font
-					(size 1.27 1.27)
-				)
-				(justify right)
-				(hide yes)
-			)
-		)
-	)
 	(global_label "PB4"
 		(shape input)
@@
 		)
 	)
-	(global_label "IR_4"
-		(shape input)
-		(at 228.6 81.28 180)
-		(fields_autoplaced yes)
-		(effects
-			(font
-				(size 1.016 1.016)
-			)
-			(justify right)
-		)
-		(property "Intersheetrefs" "${INTERSHEET_REFS}"
-			(at 222.9706 81.28 0)
-			(effects
-				(font
-					(size 1.27 1.27)
-				)
-				(justify right)
-				(hide yes)
-			)
-		)
-	)
 	(global_label "PD2"
 		(shape input)
@@
 				(hide yes)
 			)
-		)
-	)
-	(global_label "IR_3"
-		(shape input)
-		(at 215.9 81.28 180)
-		(fields_autoplaced yes)
-		(effects
-			(font
-				(size 1.016 1.016)
-			)
-			(justify right)
-		)
-		(property "Intersheetrefs" "${INTERSHEET_REFS}"
-			(at 210.2706 81.28 0)
-			(effects
-				(font
-					(size 1.27 1.27)
-				)
-				(justify right)
-				(hide yes)
-			)
