File: Hardware/mainboard/programming.kicad_sch (KiCad schematic)
At the start: 12 parts, among them J6 Conn_01x06_Socket, J7 SBH11-PBPC-D05-ST-BK, J9 USB_C_Receptacle_PowerOnly_24P, U2 AMS1117-3.3

Commit message: pushing for the evening
didnt add much, just moved things around and fixed footprints
Changed lines of the file:
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@@
 	(text "Only one of these should be plugged in at once.\n\nDo not try to power it with USB-C while programming \nwith JTAG and USB-TTL."
 		(exclude_from_sim no)
-		(at 178.308 29.972 0)
+		(at 106.172 24.384 0)
 		(effects
 			(font

Commit message: Lowkey forgot the start switch so i added that
Parts:
- C1: value C -> 100nF
- C2: value C -> 10uF
- C3, C4: value C -> 22uF
- D1, D3: value SMAZ5V1-13-F -> zener
- R1: value R_US -> 1k5
Other:
- note added: "RED"
Changed lines of the file:
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@@
+		)
+	)
+	(text "RED\n"
+		(exclude_from_sim no)
+		(at 168.656 74.676 0)
+		(effects
+			(font
+				(size 1.27 1.27)
+			)
 		)
 	)
@@
 			)
 		)
-		(property "Value" "C"
+		(property "Value" "10uF"
 			(at 107.95 71.12 90)
 			(effects
@@
 			)
 		)
-		(property "Value" "SMAZ5V1-13-F"
+		(property "Value" "zener"
 			(at 81.28 73.152 0)
 			(effects
@@
 			)
 		)
-		(property "Value" "C"
+		(property "Value" "22uF"
 			(at 114.8874 83.106 0)
 			(effects
@@
 			)
 		)
-		(property "Value" "C"
+		(property "Value" "100nF"
 			(at 95.25 71.12 90)
 			(effects
@@
 			)
 		)
-		(property "Value" "C"
+		(property "Value" "22uF"
 			(at 149.86 82.5499 0)
 			(effects
@@
 			)
 		)
-		(property "Value" "R_US"
+		(property "Value" "1k5"
 			(at 161.6234 83.868 0)
 			(effects
@@
 			)
 		)
-		(property "Value" "SMAZ5V1-13-F"
+		(property "Value" "zener"
 			(at 81.28 87.376 0)
 			(effects

Commit message: layout
worked on the layput but im actively falling asleep while working on it so im going to call it a day
Parts:
- J6: footprint Connector_PinHeader_1.00mm:PinHeader_1x06_P1.00mm_Vertical -> Connector_PinHeader_2.54mm:PinHeader_1x06_P2.54mm_Vertical
Changed lines of the file:
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@@
 			)
 		)
-		(property "Footprint" "Connector_PinHeader_1.00mm:PinHeader_1x06_P1.00mm_Vertical"
+		(property "Footprint" "Connector_PinHeader_2.54mm:PinHeader_1x06_P2.54mm_Vertical"
 			(at 31.75 31.75 0)
 			(effects

Commit message: add layer
Parts:
- removed J9: USB_C_Receptacle_PowerOnly_24P, usbc_power_only:KUSBX-SMT-CS-6-BTR_KYC, symbol Connector:USB_C_Receptacle_PowerOnly_24P
- added J8: KUSBX-SMT-CS-6-BTR, KUSBX-SMT-CS-6-BTR_KYC, symbol USB-C-PORT:KUSBX-SMT-CS-6-BTR
- J6: value Conn_01x06_Socket -> usb-ttl
- J7: value SBH11-PBPC-D05-ST-BK -> jtag
Connections:
- net 5v5_usb: now also J8.A9 (VBUS), J8.B9 (VBUS)
- net GND: now also J8.A12 (GND), J8.B12 (GND)
- no-connect marks 8 -> 7
Other:
- moved on the sheet: D3

Commit message: routed traces
Parts:
- J6: footprint Connector_PinHeader_2.54mm:PinHeader_1x06_P2.54mm_Vertical -> Connector_PinSocket_2.54mm:PinSocket_1x06_P2.54mm_Vertical
Changed lines of the file:
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@@
 			)
 		)
-		(property "Footprint" "Connector_PinHeader_2.54mm:PinHeader_1x06_P2.54mm_Vertical"
+		(property "Footprint" "Connector_PinSocket_2.54mm:PinSocket_1x06_P2.54mm_Vertical"
 			(at 31.75 31.75 0)
 			(effects

Commit message: generated gbr files
Parts:
- added TP4, TP5: TestPoint, TestPoint:TestPoint_Keystone_5019_Minature, symbol Connector:TestPoint
Connections:
- net 5v5_post_diode: now also TP4.1
- net GND: now also TP5.1
Changed lines of the file:
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@@
+	)
+	(junction
+		(at 87.63 93.98)
+		(diameter 0)
+		(color 0 0 0 0)
 	)
 	(junction
@@
 	(wire
 		(pts
-			(xy 87.63 76.2) (xy 87.63 104.14)
+			(xy 87.63 76.2) (xy 87.63 93.98)
 		)
 		(stroke
@@
 		(pts
 			(xy 146.05 77.47) (xy 146.05 76.2)
+		)
+		(stroke
+			(width 0)
+			(type default)
+		)
+	)
+	(wire
+		(pts
+			(xy 87.63 93.98) (xy 87.63 104.14)
 		)
 		(stroke
@@
 	(rectangle
 		(start 113.03 64.77)
-		(end 166.37 91.44)
+		(end 166.37 93.98)
 		(stroke
 			(width 0)
@@
 				(justify left)
 				(hide yes)
+			)
+		)
+	)
+	(symbol
+		(lib_id "Connector:TestPoint")
+		(at 87.63 93.98 270)
+		(unit 1)
+		(exclude_from_sim no)
+		(in_bom yes)
+		(on_board yes)
+		(dnp no)
+		(fields_autoplaced yes)
+		(property "Reference" "TP4"
+			(at 92.71 92.7099 90)
+			(effects
+				(font
+					(size 1.27 1.27)
+				)
+				(justify left)
+			)
+		)
+		(property "Value" "TestPoint"
+			(at 92.71 95.2499 90)
+			(effects
+				(font
+					(size 1.27 1.27)
+				)
+				(justify left)
+			)
+		)
+		(property "Footprint" "TestPoint:TestPoint_Keystone_5019_Minature"
+			(at 87.63 99.06 0)
+			(effects
+				(font
+					(size 1.27 1.27)
+				)
+				(hide yes)
+			)
+		)
+		(property "Datasheet" "~"
+			(at 87.63 99.06 0)
+			(effects
+				(font
+					(size 1.27 1.27)
+				)
+				(hide yes)
+			)
+		)
+		(property "Description" "test point"
+			(at 87.63 93.98 0)
+			(effects
+				(font
+					(size 1.27 1.27)
+				)
+				(hide yes)
+			)
+		)
+		(pin "1"
+		)
+		(instances
+			(project "mainboard"
+				(path "/5f7c2eda-1e0f-4231-89f6-49a17b370d9e/7b524a24-56f0-4a49-a03c-55156da3f2cd"
+					(reference "TP4")
+					(unit 1)
+				)
 			)
 		)
@@
 					(unit 1)
 				)
+			)
+		)
+	)
+	(symbol
+		(lib_id "Connector:TestPoint")
+		(at 146.05 87.63 180)
+		(unit 1)
+		(exclude_from_sim no)
+		(in_bom yes)
+		(on_board yes)
+		(dnp no)
+		(fields_autoplaced yes)
+		(property "Reference" "TP5"
+			(at 148.59 89.6619 0)
+			(effects
+				(font
+					(size 1.27 1.27)
+				)
+				(justify right)
+			)
+		)
+		(property "Value" "TestPoint"
+			(at 148.59 92.2019 0)
+			(effects
+				(font
+					(size 1.27 1.27)
+				)
+				(justify right)
+			)
+		)
+		(property "Footprint" "TestPoint:TestPoint_Keystone_5019_Minature"
+			(at 140.97 87.63 0)
+			(effects
+				(font
+					(size 1.27 1.27)
+				)
+				(hide yes)
+			)
+		)
+		(property "Datasheet" "~"
+			(at 140.97 87.63 0)
+			(effects
+				(font
+					(size 1.27 1.27)
+				)
+				(hide yes)
+			)
+		)
+		(property "Description" "test point"
+			(at 146.05 87.63 0)
+			(effects
+				(font
+					(size 1.27 1.27)
+				)
+				(hide yes)
+			)
+		)
+		(pin "1"
+		)
+		(instances
+			(project "mainboard"
+				(path "/5f7c2eda-1e0f-4231-89f6-49a17b370d9e/7b524a24-56f0-4a49-a03c-55156da3f2cd"
+					(reference "TP5")
+					(unit 1)
+				)
