File: Hardware/mainboard/mainboard.kicad_pcb (KiCad board)
At the start: 4 copper layers, 78 x 69.1 mm, 45 parts, among them J1 559592430, J2 status bot, J3 status eot, J4 B02B-XASK-1LFSN, J5 race start, J6 usb-ttl, J7 jtag, J8 KUSBX-SMT-CS-6-BTR, SW1 ON-BOARD, SW2 BOT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

Commit message: generated gbr files
Parts:
- added TP4: TestPoint, TestPoint:TestPoint_Keystone_5019_Minature, B.Cu at (74.9, 78.6)
- added TP5: TestPoint, TestPoint:TestPoint_Keystone_5019_Minature, F.Cu at (107.9, 86.2)
- added TP6: TestPoint, TestPoint:TestPoint_Keystone_5019_Minature, B.Cu at (83.8, 65.9)
- added TP7: TestPoint, TestPoint:TestPoint_Keystone_5019_Minature, F.Cu at (79.9, 48.1)
- added TP8: TestPoint, TestPoint:TestPoint_Keystone_5019_Minature, B.Cu at (120.6, 85.0)
- TP3: value PC11 -> TestPoint
- moved C1 5.10 mm to (82.0, 77.3)
- moved C12 5.10 mm to (118.5, 77.7)
- moved C13 5.10 mm to (126.7, 75.1)
- moved C14 5.10 mm to (101.8, 65.3)
- moved C2 5.10 mm to (82.0, 82.3)
- moved C3 5.10 mm to (87.9, 74.3)
- moved C4 5.10 mm to (93.2, 74.3)
- moved C5 5.10 mm to (93.3, 69.2)
- moved C7 5.10 mm to (117.0, 70.8)
- moved C8 5.10 mm to (117.5, 60.6)
- moved C9 5.10 mm to (104.1, 73.1)
- moved D1 5.10 mm to (74.9, 75.1)
- moved D3 5.10 mm to (74.9, 82.7)
- moved H3 5.10 mm to (67.8, 90.6)
- moved J2 5.10 mm to (66.7, 42.6)
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Routing:
- net /programming/5v5_post_diode: track 14.7 -> 19.2 mm, vias 0 -> 1
- net GND: track 28.4 -> 30.9 mm
Other:
- board text added: "5v5"

Commit message: gbr files
ordered pcbs
Parts:
- J8: footprint BIG LIBRARY:usb-c2 -> usbc attempt 3:2171750001_MOL
- moved G*** 6.85 mm to (91.4, 61.1)
- moved R1 2.20 mm to (90.5, 92.1)
- moved SW2 2.20 mm to (135.8, 77.2)
- moved TP8 2.20 mm to (122.4, 86.1)
- moved U1 2.20 mm to (132.3, 68.0)
- moved J1 2.20 mm to (95.4, 37.2)
- moved U3 2.20 mm to (115.3, 61.8)
- moved H2 2.20 mm to (138.4, 31.8)
- moved C3 2.20 mm to (89.8, 75.4)
- moved C4 2.20 mm to (95.0, 75.5)
- moved D1 2.20 mm to (76.7, 76.2)
- moved D3 2.20 mm to (76.7, 83.9)
- moved H4 2.20 mm to (138.4, 91.7)
- moved J2 2.20 mm to (68.6, 43.8)
- moved J5 2.20 mm to (131.8, 39.0)
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Routing:
- net PC9: track 37.9 -> 37.2 mm
- net PB2: track 66.9 -> 67.4 mm
- net /stm/BOOT0: track 20.8 -> 20.3 mm
- net GND: track 30.9 -> 30.4 mm
